File: TTB KiCAD FIles.kicad_pcb (KiCad board)
At the start: 2 copper layers, 174.2 x 86.7 mm, 5 parts, among them J1 PJ-102A, U1 Relay Control Module, U2 ESP32 Module, U3 Motor Driver Module, U4 Pololu_Voltage_Regulator

Commit message: Updates
Parts:
- added J2: Conn_01x03_Pin, Connector_PinHeader_2.54mm:PinHeader_1x03_P2.54mm_Vertical, F.Cu at (141.8, 127.7)
- U1: value Relay Control Module -> Relay Module
- U3: value Motor Driver Module -> Motor Driver
- U4: value Pololu_Voltage_Regulator -> Voltage Regulator
Routing:
- net +5V: track 34.4 -> 75.3 mm
- net +12V: track 355.8 -> 368.1 mm
- net Net-(U2-3V3): track 17.7 -> 19.7 mm
- net Net-(U2-D23): track 20.8 -> 22.8 mm
- net Net-(U1-IN3): track 24.9 -> 26.4 mm
- net Net-(U1-IN2): track 22.4 -> 23.9 mm
- net Net-(U1-IN1): track 19.9 -> 21.1 mm
Other:
- board text added: "12V"
- board text added: "5V"
- board text added: "GND"
